Commit message: 1. Modified pid control for doggo_bot ros_controller for stable simulation. 2. Added moveit python command code for moveit interface control. 3. Changed effort magnitude for doggo_robot.urdf.

File: src/doggo_robot/urdf/doggo_robot.urdf (robot description, URDF)
Before this commit: robot doggo_robot, 17 links, 16 joints
Joints:
- joint BackLeftJoint1: limit lower=-3.14 upper=3.14 effort=1 velocity=1 -> lower=-3.14 upper=3.14 effort=10 velocity=1
- joint BackLeftJoint2: limit lower=-3.14 upper=3.14 effort=1 velocity=1 -> lower=-3.14 upper=3.14 effort=10 velocity=1
- joint BackLeftJoint3: limit lower=-3.14 upper=3.14 effort=1 velocity=1 -> lower=-3.14 upper=3.14 effort=10 velocity=1
- joint BackRightJoint1: limit lower=-3.14 upper=3.14 effort=1 velocity=1 -> lower=-3.14 upper=3.14 effort=10 velocity=1
- joint BackRightJoint2: limit lower=-3.14 upper=3.14 effort=1 velocity=1 -> lower=-3.14 upper=3.14 effort=10 velocity=1
- joint BackRightJoint3: limit lower=-3.14 upper=3.14 effort=1 velocity=1 -> lower=-3.14 upper=3.14 effort=10 velocity=1
- joint FrontLeftJoint1: limit lower=-3.14 upper=3.14 effort=1 velocity=1 -> lower=-3.14 upper=3.14 effort=10 velocity=1
- joint FrontLeftJoint2: limit lower=-3.14 upper=3.14 effort=1 velocity=1 -> lower=-3.14 upper=3.14 effort=10 velocity=1
- joint FrontLeftJoint3: limit lower=-3.14 upper=3.14 effort=1 velocity=1 -> lower=-3.14 upper=3.14 effort=10 velocity=1
- joint FrontRightJoint1: limit lower=-3.14 upper=3.14 effort=1 velocity=1 -> lower=-3.14 upper=3.14 effort=10 velocity=1
- joint FrontRightJoint2: limit lower=-3.14 upper=3.14 effort=1 velocity=1 -> lower=-3.14 upper=3.14 effort=10 velocity=1
- joint FrontRightJoint3: limit lower=-3.14 upper=3.14 effort=1 velocity=1 -> lower=-3.14 upper=3.14 effort=10 velocity=1

Commit message: 1. Integrated stanford robot to gazebo 2. changed parameter to stable gazebo simulation

File: src/doggo_robot/urdf/doggo_robot.urdf (robot description, URDF)
Before this commit: robot doggo_robot, 18 links, 17 joints
Joints:
- joint BackLeftJoint1: limit lower=-3.14 upper=3.14 effort=15 velocity=1 -> lower=-3.14 upper=3.14 effort=15 velocity=5
- joint BackLeftJoint2: limit lower=-3.14 upper=3.14 effort=15 velocity=1 -> lower=-3.14 upper=3.14 effort=15 velocity=5
- joint BackLeftJoint3: limit lower=-3.14 upper=3.14 effort=15 velocity=1 -> lower=-3.14 upper=3.14 effort=15 velocity=5
- joint BackRightJoint1: limit lower=-3.14 upper=3.14 effort=15 velocity=1 -> lower=-3.14 upper=3.14 effort=15 velocity=5
- joint BackRightJoint2: limit lower=-3.14 upper=3.14 effort=15 velocity=1 -> lower=-3.14 upper=3.14 effort=15 velocity=5
- joint BackRightJoint3: limit lower=-3.14 upper=3.14 effort=15 velocity=1 -> lower=-3.14 upper=3.14 effort=15 velocity=5
- joint FrontLeftJoint1: limit lower=-3.14 upper=3.14 effort=15 velocity=1 -> lower=-3.14 upper=3.14 effort=15 velocity=5
- joint FrontLeftJoint2: limit lower=-3.14 upper=3.14 effort=15 velocity=1 -> lower=-3.14 upper=3.14 effort=15 velocity=5
- joint FrontLeftJoint3: limit lower=-3.14 upper=3.14 effort=15 velocity=1 -> lower=-3.14 upper=3.14 effort=15 velocity=5
- joint FrontRightJoint1: limit lower=-3.14 upper=3.14 effort=15 velocity=1 -> lower=-3.14 upper=3.14 effort=15 velocity=5
- joint FrontRightJoint2: limit lower=-3.14 upper=3.14 effort=15 velocity=1 -> lower=-3.14 upper=3.14 effort=15 velocity=5
- joint FrontRightJoint3: limit lower=-3.14 upper=3.14 effort=15 velocity=1 -> lower=-3.14 upper=3.14 effort=15 velocity=5

Commit message: Modify the robot such that it is able to walk, still experiencing sliding issue

File: src/doggo_robot/urdf/doggo_robot.urdf (robot description, URDF)
Before this commit: robot doggo_robot, 18 links, 17 joints
Links:
- removed link world
- link BackLeftLink2: mass 0.45685 -> 0.4003
- link BackLeftLink3: mass 0.35095 -> 0.20957
- link BackRightLink2: mass 0.45685 -> 0.4003
- link BackRightLink3: mass 0.35095 -> 0.20957
- link FrontLeftLink1: mass 0.23902 -> 0.239017817769067
- link FrontLeftLink2: mass 0.45685 -> 0.4003
- link FrontLeftLink3: mass 0.35095 -> 0.20957
- link FrontRightLink2: mass 0.45685 -> 0.4003
- link FrontRightLink3: mass 0.35095 -> 0.20957
- link base_link: mass 8.7429 -> 1
Joints:
- removed joint world_link_to_base_link
- joint BackLeftJoint1: limit lower=-3.14 upper=3.14 effort=15 velocity=5 -> lower=-3.14 upper=3.14 effort=10 velocity=0.8; origin xyz=0.09 0.22 0.0505413918665349 rpy=-1.5707963267949 0 0 -> xyz=-0.22 0.09 0.00054139 rpy=1.5708 0 1.5708
- joint BackLeftJoint2: axis 0 0 -1 -> 0 0 1; limit lower=-3.14 upper=3.14 effort=15 velocity=5 -> lower=-3.14 upper=3.14 effort=10 velocity=0.8; origin xyz=0.07 0 0 rpy=1.5707963267949 0 1.5707963267949 -> xyz=0.07 0 0 rpy=-1.5708 0 -1.5708
- joint BackLeftJoint3: limit lower=-3.14 upper=3.14 effort=15 velocity=5 -> lower=-3.14 upper=3.14 effort=10 velocity=0.8; origin xyz=0.15 0 0.0649999999999999 rpy=0 0 0 -> xyz=0.15 0 0 rpy=0 0 0
- joint BackRightJoint1: axis 0 0 -1 -> 0 0 1; limit lower=-3.14 upper=3.14 effort=15 velocity=5 -> lower=-3.14 upper=3.14 effort=10 velocity=0.8; origin xyz=-0.09 0.22 0.0505413918665349 rpy=1.5707963267949 0 3.14159265358979 -> xyz=-0.22 -0.09 0.00054139 rpy=-1.5708 0 -1.5708
- joint BackRightJoint2: axis 0 0 -1 -> 0 0 1; limit lower=-3.14 upper=3.14 effort=15 velocity=5 -> lower=-3.14 upper=3.14 effort=10 velocity=0.8; origin xyz=0.07 0 0 rpy=-1.5707963267949 0 -1.5707963267949 -> xyz=0.07 0 0 rpy=-1.5708 0 1.5708
- joint BackRightJoint3: axis 0 0 -1 -> 0 0 1; limit lower=-3.14 upper=3.14 effort=15 velocity=5 -> lower=-3.14 upper=3.14 effort=10 velocity=0.8; origin xyz=0.15 0 0.065 rpy=3.14159265358979 0 0 -> xyz=0.15 0 0 rpy=0 0 0
- joint FrontLeftJoint1: axis 0 0 -1 -> 0 0 1; limit lower=-3.14 upper=3.14 effort=15 velocity=5 -> lower=-3.14 upper=3.14 effort=10 velocity=0.8; origin xyz=0.09 -0.22 0.0505413918665349 rpy=1.5707963267949 0.00226227152123116 0 -> xyz=0.22 0.09 0.00054139 rpy=1.5708 0.0022623 1.5708
- joint FrontLeftJoint2: axis 0 0 -1 -> 0 0 1; limit lower=-3.14 upper=3.14 effort=15 velocity=5 -> lower=-3.14 upper=3.14 effort=10 velocity=0.8; origin xyz=0.0699999999999998 0 0 rpy=-1.5707963267949 0 -1.5707963267949 -> xyz=0.07 0 0 rpy=-1.5708 0 -1.5708
- joint FrontLeftJoint3: limit lower=-3.14 upper=3.14 effort=15 velocity=5 -> lower=-3.14 upper=3.14 effort=10 velocity=0.8; origin xyz=0.15 0 0.0650000000000001 rpy=0 0 0 -> xyz=0.15 0 0 rpy=0 0 0
- joint FrontRightJoint1: limit lower=-3.14 upper=3.14 effort=15 velocity=5 -> lower=-3.14 upper=3.14 effort=10 velocity=0.8; origin xyz=-0.0899999999999993 -0.22 0.0505413918665352 rpy=-1.5707963267949 0.00403021498393773 -3.14159265358979 -> xyz=0.22 -0.09 0.00054139 rpy=-1.5708 0.0040302 -1.5708
- joint FrontRightJoint2: axis 0 0 -1 -> 0 0 1; limit lower=-3.14 upper=3.14 effort=15 velocity=5 -> lower=-3.14 upper=3.14 effort=10 velocity=0.8; origin xyz=0.0700000000000005 0 0 rpy=1.5707963267949 0 1.5707963267949 -> xyz=0.07 0 0 rpy=-1.5708 0 1.5708
- joint FrontRightJoint3: limit lower=-3.14 upper=3.14 effort=15 velocity=5 -> lower=-3.14 upper=3.14 effort=10 velocity=0.8; origin xyz=0.15 0 0.065 rpy=0 0 0 -> xyz=0.15 0 0 rpy=0 0 0
